File: footswitch-pcb/footswitch-pcb.kicad_sch (KiCad schematic)
At the start: 6 parts, among them J2 Conn_01x02_Female, SW3 SW_SPST, U1 SeeeduinoXIAO

Commit message: PCB Update
Parts:
- removed J1: (no value), symbol Connector:Conn_01x02_Female
- removed J2: Conn_01x02_Female, symbol Connector:Conn_01x02_Female
- removed SW1: (no value), symbol Switch:SW_SPST
- removed SW3: SW_SPST, symbol Switch:SW_SPST
- added D1: (no value), symbol LED:WS2812B
- added D2: (no value), symbol Device:LED_RKGB
- added J1, J4: (no value), symbol Connector:Conn_01x02_Male
- added J2, J3, J5: (no value), symbol Connector:Conn_01x01_Male
- added R1: (no value), symbol Device:R
- added R2, R3: R, symbol Device:R
- added SW1: (no value), symbol Switch:SW_DIP_x03
- added SW3: (no value), Button_Switch_THT:SW_Tactile_SPST_Angled_PTS645Vx39-2LFS, symbol Switch:SW_Push
- SW2: value (none) -> SW_BLUETOOTH; footprint (none) -> Button_Switch_THT:SW_Tactile_SPST_Angled_PTS645Vx39-2LFS
Connections:
- net GND: now also SW2.2, D2.2 (K), J1.1 (Pin_1), SW1.1, SW1.2, SW1.3, SW3.2; no longer SW2.1
- net PIN_BT: now reaches U1.1 (PA02_A0_D0)
- net PIN_BT: now also SW2.1
- net PIN_LAYER2: now reaches U1.10 (PA5_A9_D9_MISO)
- net PIN_LAYER2: now also SW1.5
- net PIN_LAYER1: now reaches U1.11 (PA6_A10_D10_MOSI)
- net PIN_LAYER1: now also SW1.6
- net PIN_LEDR: now reaches U1.2 (PA4_A1_D1)
- net PIN_LEDR: now also R3.2
- net PIN_LEDG: now reaches U1.3 (PA10_A2_D2)
- net PIN_LEDG: now also R2.2; no longer SW2.2
- net PIN_LEDB: now reaches U1.4 (PA11_A3_D3)
- net PIN_LEDB: now also R1.2
- net PIN_PEDAL: now reaches U1.8 (PB09_A7_D7_RX)
- net PIN_PEDAL: now also J1.2 (Pin_2)
- net PIN_LAYER3: now reaches U1.9 (PA7_A8_D8_SCK)
- net PIN_LAYER3: now also SW1.4
- new net: J3.1 (Pin_1), SW3.1
- new net: J2.1 (Pin_1), J4.2 (Pin_2)
- new net: J4.1 (Pin_1), J5.1 (Pin_1)
- new net: D2.1 (RA), R3.1
- new net: D2.3 (GA), R2.1
- new net: D2.4 (BA), R1.1
- no-connect marks 15 -> 14
Other:
- moved on the sheet: SW2

Commit message: PCB update
Parts:
- removed SW3: (no value), Button_Switch_THT:SW_Tactile_SPST_Angled_PTS645Vx39-2LFS, symbol Switch:SW_Push
- added SW3: SW_SPDT, Button_Switch_THT:SW_Slide_1P2T_CK_OS102011MS2Q, symbol Switch:SW_SPDT
- D1: value (none) -> WS2812B; footprint (none) -> LED_SMD:LED_WS2812B_PLCC4_5.0x5.0mm_P3.2mm
- D2: value (none) -> LED_RKGB; footprint (none) -> LED_THT:LED_D5.0mm-4_RGB_Wide_Pins
- J1: value (none) -> Conn_Pedal; footprint (none) -> Connector_JST:JST_XH_B2B-XH-A_1x02_P2.50mm_Vertical
- J2: value (none) -> Solder_Pad_BAT+; footprint (none) -> TestPoint:TestPoint_Pad_3.0x3.0mm
- J3: value (none) -> Solder_Pad_Reset; footprint (none) -> TestPoint:TestPoint_Pad_3.0x3.0mm
- J4: value (none) -> Conn_01x02_Male; footprint (none) -> Connector_JST:JST_XH_S2B-XH-A-1_1x02_P2.50mm_Horizontal
- J5: value (none) -> Solder_Pad_BAT-; footprint (none) -> TestPoint:TestPoint_Pad_3.0x3.0mm
- R1: value (none) -> R; footprint (none) -> Resistor_SMD:R_0402_1005Metric_Pad0.72x0.64mm_HandSolder
- R2, R3: footprint (none) -> Resistor_SMD:R_0402_1005Metric_Pad0.72x0.64mm_HandSolder
- SW1: value (none) -> SW_DIP_x03; footprint (none) -> Button_Switch_THT:SW_DIP_SPSTx03_Slide_6.7x9.18mm_W7.62mm_P2.54mm_LowProfile
Connections:
- net GND: now also SW3.3 (C)
- net at J3.1 (Pin_1): now also SW3.2 (B)
- no-connect marks 14 -> 15
Changed lines of the file:
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@@
   (no_connect (at 120.65 100.33))
   (no_connect (at 127 55.88))
+  (no_connect (at 135.89 33.02))
   (no_connect (at 144.78 100.33))
   (no_connect (at 140.97 100.33))
@@
     (in_bom yes) (on_board yes) (fields_autoplaced)
     (property "Reference" "J1" (id 0) (at 51.435 97.756 0))
-    (property "Value" "" (id 1) (at 51.435 95.2191 0))
-    (property "Footprint" "" (id 2) (at 52.07 93.98 0)
+    (property "Value" "Conn_Pedal" (id 1) (at 51.435 95.2191 0))
+    (property "Footprint" "Connector_JST:JST_XH_B2B-XH-A_1x02_P2.50mm_Vertical" (id 2) (at 52.07 93.98 0)
       (effects (font (size 1.27 1.27)) hide)
     )
@@
     (in_bom yes) (on_board yes) (fields_autoplaced)
     (property "Reference" "D1" (id 0) (at 207.1559 86.7116 0))
-    (property "Value" "" (id 1) (at 207.1559 89.2485 0))
-    (property "Footprint" "" (id 2) (at 198.12 97.79 0)
+    (property "Value" "WS2812B" (id 1) (at 207.1559 89.2485 0))
+    (property "Footprint" "LED_SMD:LED_WS2812B_PLCC4_5.0x5.0mm_P3.2mm" (id 2) (at 198.12 97.79 0)
       (effects (font (size 1.27 1.27)) (justify left top) hide)
     )
@@
     (pin "4")
   )
-  (symbol (lib_id "power:GND") (at 135.89 35.56 0) (unit 1)
-    (in_bom yes) (on_board yes) (fields_autoplaced)
-    (property "Reference" "#PWR0103" (id 0) (at 135.89 41.91 0)
-      (effects (font (size 1.27 1.27)) hide)
-    )
-    (property "Value" "GND" (id 1) (at 137.795 37.2638 0)
+  (symbol (lib_id "power:GND") (at 135.89 38.1 0) (unit 1)
+    (in_bom yes) (on_board yes) (fields_autoplaced)
+    (property "Reference" "#PWR0103" (id 0) (at 135.89 44.45 0)
+      (effects (font (size 1.27 1.27)) hide)
+    )
+    (property "Value" "GND" (id 1) (at 137.795 39.8038 0)
       (effects (font (size 1.27 1.27)) (justify left))
     )
-    (property "Footprint" "" (id 2) (at 135.89 35.56 0)
-      (effects (font (size 1.27 1.27)) hide)
-    )
-    (property "Datasheet" "" (id 3) (at 135.89 35.56 0)
+    (property "Footprint" "" (id 2) (at 135.89 38.1 0)
+      (effects (font (size 1.27 1.27)) hide)
+    )
+    (property "Datasheet" "" (id 3) (at 135.89 38.1 0)
       (effects (font (size 1.27 1.27)) hide)
     )
@@
     (in_bom yes) (on_board yes)
     (property "Reference" "J3" (id 0) (at 121.92 36.83 90))
-    (property "Value" "" (id 1) (at 114.3 39.37 90))
-    (property "Footprint" "" (id 2) (at 125.73 40.64 0)
+    (property "Value" "Solder_Pad_Reset" (id 1) (at 114.3 39.37 90))
+    (property "Footprint" "TestPoint:TestPoint_Pad_3.0x3.0mm" (id 2) (at 125.73 40.64 0)
       (effects (font (size 1.27 1.27)) hide)
     )
@@
     (in_bom yes) (on_board yes)
     (property "Reference" "J2" (id 0) (at 114.3 107.95 0))
-    (property "Value" "" (id 1) (at 113.03 110.49 0))
-    (property "Footprint" "" (id 2) (at 113.03 113.03 0)
+    (property "Value" "Solder_Pad_BAT+" (id 1) (at 113.03 110.49 0))
+    (property "Footprint" "TestPoint:TestPoint_Pad_3.0x3.0mm" (id 2) (at 113.03 113.03 0)
       (effects (font (size 1.27 1.27)) hide)
     )
@@
       (effects (font (size 1.27 1.27)) (justify right))
     )
-    (property "Value" "" (id 1) (at 132.7912 116.0022 0)
+    (property "Value" "Conn_01x02_Male" (id 1) (at 132.7912 116.0022 0)
       (effects (font (size 1.27 1.27)) (justify right))
     )
-    (property "Footprint" "" (id 2) (at 132.08 115.57 0)
+    (property "Footprint" "Connector_JST:JST_XH_S2B-XH-A-1_1x02_P2.50mm_Horizontal" (id 2) (at 132.08 115.57 0)
       (effects (font (size 1.27 1.27)) hide)
     )
@@
     (in_bom yes) (on_board yes) (fields_autoplaced)
     (property "Reference" "SW1" (id 0) (at 63.5 63.6102 0))
-    (property "Value" "" (id 1) (at 63.5 66.1471 0))
-    (property "Footprint" "" (id 2) (at 63.5 74.93 0)
+    (property "Value" "SW_DIP_x03" (id 1) (at 63.5 66.1471 0))
+    (property "Footprint" "Button_Switch_THT:SW_DIP_SPSTx03_Slide_6.7x9.18mm_W7.62mm_P2.54mm_LowProfile" (id 2) (at 63.5 74.93 0)
       (effects (font (size 1.27 1.27)) hide)
     )
@@
     (in_bom yes) (on_board yes)
     (property "Reference" "J5" (id 0) (at 114.3 116.84 0))
-    (property "Value" "" (id 1) (at 113.03 119.38 0))
-    (property "Footprint" "" (id 2) (at 113.03 115.57 0)
+    (property "Value" "Solder_Pad_BAT-" (id 1) (at 113.03 119.38 0))
+    (property "Footprint" "TestPoint:TestPoint_Pad_3.0x3.0mm" (id 2) (at 113.03 115.57 0)
       (effects (font (size 1.27 1.27)) hide)
     )
@@
     (property "Reference" "R3" (id 0) (at 191.77 66.4042 90))
     (property "Value" "R" (id 1) (at 191.77 68.9411 90))
-    (property "Footprint" "" (id 2) (at 191.77 69.342 90)
+    (property "Footprint" "Resistor_SMD:R_0402_1005Metric_Pad0.72x0.64mm_HandSolder" (id 2) (at 191.77 69.342 90)
       (effects (font (size 1.27 1.27)) hide)
     )
@@
     (pin "1")
     (pin "2")
+  )
+  (symbol (lib_id "Switch:SW_SPDT") (at 130.81 35.56 0) (unit 1)
+    (in_bom yes) (on_board yes) (fields_autoplaced)
+    (property "Reference" "SW3" (id 0) (at 130.81 27.94 0))
+    (property "Value" "SW_SPDT" (id 1) (at 130.81 30.48 0))
+    (property "Footprint" "Button_Switch_THT:SW_Slide_1P2T_CK_OS102011MS2Q" (id 2) (at 130.81 35.56 0)
+      (effects (font (size 1.27 1.27)) hide)
+    )
+    (property "Datasheet" "~" (id 3) (at 130.81 35.56 0)
+      (effects (font (size 1.27 1.27)) hide)
+    )
+    (pin "1")
+    (pin "2")
+    (pin "3")
   )
   (symbol (lib_id "Device:R") (at 191.77 66.04 270) (unit 1)
@@
     (property "Reference" "R2" (id 0) (at 191.77 61.3242 90))
     (property "Value" "R" (id 1) (at 191.77 63.8611 90))
-    (property "Footprint" "" (id 2) (at 191.77 64.262 90)
+    (property "Footprint" "Resistor_SMD:R_0402_1005Metric_Pad0.72x0.64mm_HandSolder" (id 2) (at 191.77 64.262 90)
       (effects (font (size 1.27 1.27)) hide)
     )
@@
     (pin "1")
   )
-  (symbol (lib_id "Switch:SW_Push") (at 130.81 35.56 0) (unit 1)
-    (in_bom yes) (on_board yes) (fields_autoplaced)
-    (property "Reference" "SW3" (id 0) (at 130.81 28.9392 0))
-    (property "Value" "" (id 1) (at 130.81 31.4761 0))
-    (property "Footprint" "Button_Switch_THT:SW_Tactile_SPST_Angled_PTS645Vx39-2LFS" (id 2) (at 130.81 30.48 0)
-      (effects (font (size 1.27 1.27)) hide)
-    )
-    (property "Datasheet" "~" (id 3) (at 130.81 30.48 0)
-      (effects (font (size 1.27 1.27)) hide)
-    )
-    (pin "1")
-    (pin "2")
-  )
   (symbol (lib_id "Device:LED_RKGB") (at 200.66 66.04 180) (unit 1)
     (in_bom yes) (on_board yes) (fields_autoplaced)
     (property "Reference" "D2" (id 0) (at 200.66 54.7202 0))
-    (property "Value" "" (id 1) (at 200.66 57.2571 0))
-    (property "Footprint" "" (id 2) (at 200.66 64.77 0)
+    (property "Value" "LED_RKGB" (id 1) (at 200.66 57.2571 0))
+    (property "Footprint" "LED_THT:LED_D5.0mm-4_RGB_Wide_Pins" (id 2) (at 200.66 64.77 0)
       (effects (font (size 1.27 1.27)) hide)
     )
@@
     (in_bom yes) (on_board yes) (fields_autoplaced)
     (property "Reference" "R1" (id 0) (at 191.77 56.2442 90))
-    (property "Value" "" (id 1) (at 191.77 58.7811 90))
-    (property "Footprint" "" (id 2) (at 191.77 59.182 90)
+    (property "Value" "R" (id 1) (at 191.77 58.7811 90))
+    (property "Footprint" "Resistor_SMD:R_0402_1005Metric_Pad0.72x0.64mm_HandSolder" (id 2) (at 191.77 59.182 90)
       (effects (font (size 1.27 1.27)) hide)
     )
@@
       (reference "SW2") (unit 1) (value "SW_BLUETOOTH") (footprint "Button_Switch_THT:SW_Tactile_SPST_Angled_PTS645Vx39-2LFS")
     )
-    (path "/cc897e40-1e64-4f22-a40c-c00bcfcf8093"
-      (reference "SW3") (unit 1) (value "SW_RESET") (footprint "Button_Switch_THT:SW_Tactile_SPST_Angled_PTS645Vx39-2LFS")
+    (path "/be1dcc1f-57da-4659-b5f0-c69595297af6"
+      (reference "SW3") (unit 1) (value "SW_SPDT") (footprint "Button_Switch_THT:SW_Slide_1P2T_CK_OS102011MS2Q")
     )
     (path "/1d6bc926-0438-4b17-a675-0536bdc82233"

Commit message: PCB Update
Parts:
- removed D1: WS2812B, LED_SMD:LED_WS2812B_PLCC4_5.0x5.0mm_P3.2mm, symbol LED:WS2812B
- removed SW3: SW_SPDT, Button_Switch_THT:SW_Slide_1P2T_CK_OS102011MS2Q, symbol Switch:SW_SPDT
- added BTN_RESET1: BTN_RESET, Button_Switch_THT:SW_PUSH_6mm_H7.3mm, symbol Switch:SW_Push
- added SW_EN1: SW_ENABLE, Button_Switch_THT:SW_Slide_1P2T_CK_OS102011MS2Q, symbol Switch:SW_SPDT
- BTN_BT1: renamed from SW2; value SW_BLUETOOTH -> BTN_BLUETOOTH
- Pedal1: renamed from J1; footprint Connector_JST:JST_XH_B2B-XH-A_1x02_P2.50mm_Vertical -> (none)
- renumbered R3 to B1, J2 to BAT+1, J5 to BAT-1, J4 to BAT1, SW1 to DIP_MODE1, R2 to G1, J3 to RES1
Connections:
- net GND: now also BTN_RESET1.2
- net PIN_LAYER1: now also DIP_MODE1.4, U1.10 (PA5_A9_D9_MISO); no longer DIP_MODE1.6, U1.11 (PA6_A10_D10_MOSI)
- net PIN_LAYER2: now also U1.9 (PA7_A8_D8_SCK); no longer U1.10 (PA5_A9_D9_MISO)
- net PIN_LAYER3: now also DIP_MODE1.6, U1.8 (PB09_A7_D7_RX); no longer DIP_MODE1.4, U1.9 (PA7_A8_D8_SCK)
- net PIN_PEDAL: now also U1.11 (PA6_A10_D10_MOSI); no longer U1.8 (PB09_A7_D7_RX)
- net at RES1.1 (Pin_1): now also BTN_RESET1.1
- net at BAT+1.1 (Pin_1): now also SW_EN1.2 (B); no longer BAT1.2 (Pin_2)
- new net: BAT1.2 (Pin_2), SW_EN1.3 (C)
- no-connect marks 15 -> 14
Other:
- moved on the sheet: BAT1, Pedal1, RES1

Commit message: Comments in keymap, power MOSFET in schematic
Parts:
- added Q?: (no value), symbol Transistor_FET:BUK7880-55A
- BAT1: value Conn_01x02_Male -> (none)
- Pedal1: footprint (none) -> Connector_PinHeader_2.54mm:PinHeader_1x02_P2.54mm_Horizontal
Connections:
- net GND: now also BAT1.1 (Pin_1), SW_EN1.1 (A), Q?.2 (D), Q?.3 (S)
- net 5V_USB: now reaches U1.14 (5V)
- net 5V_USB: now also Q?.1 (G)
- net at SW_EN1.2 (B): now also BAT-1.1 (Pin_1); no longer BAT+1.1 (Pin_1)
- net at SW_EN1.3 (C): no longer BAT1.2 (Pin_2)
- new net: BAT+1.1 (Pin_1), BAT1.2 (Pin_2)
- no-connect marks 14 -> 13
Other:
- note added: "Drain"
- note added: "Gate"
- note added: "Source"
- moved on the sheet: BAT+1, BAT-1, BAT1, SW_EN1

Commit message: MOSFET?
Parts:
- removed BAT-1: Solder_Pad_BAT-, TestPoint:TestPoint_Pad_3.0x3.0mm, symbol Connector:Conn_01x01_Male
- added R2: 100, Resistor_SMD:R_0402_1005Metric_Pad0.72x0.64mm_HandSolder, symbol Device:R
- added R3: 10k, Resistor_SMD:R_0402_1005Metric_Pad0.72x0.64mm_HandSolder, symbol Device:R
- BAT1: value (none) -> Battery Connector
- Q1: renamed from Q?; value (none) -> BUK7880-55A; footprint (none) -> Package_TO_SOT_SMD:SOT-223-3_TabPin2
Connections:
- net 5V_USB: now also R2.1; no longer Q1.1 (G)
- net GND: now also SW_EN1.3 (C), R3.1; no longer BAT1.1 (Pin_1), DIP_MODE1.1, DIP_MODE1.2, DIP_MODE1.3, Q1.2 (D), SW_EN1.1 (A)
- net at SW_EN1.2 (B): now also BAT1.1 (Pin_1), Q1.2 (D)
- new net: Q1.1 (G), R2.2, R3.2
- new net GNDS: DIP_MODE1.1, DIP_MODE1.2, DIP_MODE1.3
Other:
- moved on the sheet: BAT+1, BAT1, Q1, SW_EN1

Commit message: THT Pogo Pins
Parts:
- removed BAT+1: Solder_Pad_BAT+, TestPoint:TestPoint_Pad_3.0x3.0mm, symbol Connector:Conn_01x01_Male
- removed RES1: Solder_Pad_Reset, TestPoint:TestPoint_Pad_3.0x3.0mm, symbol Connector:Conn_01x01_Male
Connections:
- net 5V_USB: now also R2.2; no longer R2.1
- net PIN_BT: now also U1.11 (PA6_A10_D10_MOSI); no longer U1.1 (PA02_A0_D0)
- net PIN_LAYER1: now also U1.5 (PA8_A4_D4_SDA); no longer U1.10 (PA5_A9_D9_MISO)
- net PIN_LAYER2: now also U1.6 (PA9_A5_D5_SCL); no longer U1.9 (PA7_A8_D8_SCK)
- net PIN_LAYER3: now also U1.7 (PB08_A6_D6_TX); no longer U1.8 (PB09_A7_D7_RX)
- net PIN_LEDB: now also R1.1, U1.3 (PA10_A2_D2); no longer R1.2, U1.4 (PA11_A3_D3)
- net PIN_LEDG: now also G1.1, U1.2 (PA4_A1_D1); no longer G1.2, U1.3 (PA10_A2_D2)
- net PIN_LEDR: now also U1.1 (PA02_A0_D0); no longer U1.2 (PA4_A1_D1)
- net PIN_PEDAL: now also U1.4 (PA11_A3_D3); no longer U1.11 (PA6_A10_D10_MOSI)
- net RESET: now reaches U1.17 (RESET)
- net RESET: now also BTN_RESET1.1
- net BAT+: now reaches U1.22 (BAT+)
- net BAT+: now also BAT1.2 (Pin_2)
- net at Q1.1 (G), R3.2: now also R2.1; no longer R2.2
- net at D2.3 (GA): now also G1.2; no longer G1.1
- net at D2.4 (BA): now also R1.2; no longer R1.1
- no-connect marks 13 -> 11
Other:
- moved on the sheet: G1, R1, R2
