File: footswitch-pcb/footswitch-pcb.kicad_sch (KiCad schematic)
At the start: 14 parts, among them Q1 BUK7880-55A, U1 SeeeduinoXIAO

Commit message: v3
Parts:
- B1, G1, R1, R2, R3: footprint Resistor_SMD:R_0402_1005Metric_Pad0.72x0.64mm_HandSolder -> (none)
Connections:
- net PIN_LEDB: now also B1.2, U1.10 (PA5_A9_D9_MISO); no longer R1.1, U1.3 (PA10_A2_D2)
- net PIN_LEDG: now also U1.9 (PA7_A8_D8_SCK); no longer U1.2 (PA4_A1_D1)
- net PIN_LEDR: now also R1.1, U1.8 (PB09_A7_D7_RX); no longer B1.2, U1.1 (PA02_A0_D0)
- net at B1.1: now also D2.4 (BA); no longer D2.1 (RA)
- net at R1.2: now also D2.1 (RA); no longer D2.4 (BA)
Other:
- moved on the sheet: D2
Changed lines of the file:
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@@
   )
   (no_connect (at 86.36 151.13))
-  (no_connect (at 152.4 86.36))
-  (no_connect (at 152.4 82.55))
-  (no_connect (at 152.4 90.17))
   (no_connect (at 152.4 74.93))
   (no_connect (at 124.46 100.33))
@@
   (no_connect (at 123.19 55.88))
   (no_connect (at 130.81 55.88))
+  (no_connect (at 110.49 67.31))
+  (no_connect (at 110.49 71.12))
+  (no_connect (at 110.49 74.93))
   (wire (pts (xy 58.42 139.7) (xy 58.42 135.89))
     (stroke (width 0) (type default) (color 0 0 0 0))
@@
   (global_label "PIN_LEDG" (shape input) (at 187.96 66.04 180) (fields_autoplaced)
     (effects (font (size 1.27 1.27)) (justify right))
-    (property "Intersheet References" "${INTERSHEET_REFS}" (id 0) (at 176.6569 65.9606 0)
-      (effects (font (size 1.27 1.27)) (justify right) hide)
-    )
-  )
-  (global_label "PIN_LEDB" (shape input) (at 187.96 60.96 180) (fields_autoplaced)
-    (effects (font (size 1.27 1.27)) (justify right))
-    (property "Intersheet References" "${INTERSHEET_REFS}" (id 0) (at 176.6569 60.8806 0)
+    (property "Intersheet References" "${INTERSHEET_REFS}" (id 0) (at 176.6569 66.1194 0)
+      (effects (font (size 1.27 1.27)) (justify right) hide)
+    )
+  )
+  (global_label "PIN_LEDB" (shape input) (at 187.96 71.12 180) (fields_autoplaced)
+    (effects (font (size 1.27 1.27)) (justify right))
+    (property "Intersheet References" "${INTERSHEET_REFS}" (id 0) (at 176.6569 71.1994 0)
       (effects (font (size 1.27 1.27)) (justify right) hide)
     )
@@
     )
   )
-  (global_label "PIN_LEDR" (shape input) (at 110.49 67.31 180) (fields_autoplaced)
-    (effects (font (size 1.27 1.27)) (justify right))
-    (property "Intersheet References" "${INTERSHEET_REFS}" (id 0) (at 99.1869 67.2306 0)
-      (effects (font (size 1.27 1.27)) (justify right) hide)
+  (global_label "PIN_LEDR" (shape input) (at 152.4 90.17 0) (fields_autoplaced)
+    (effects (font (size 1.27 1.27)) (justify left))
+    (property "Intersheet References" "${INTERSHEET_REFS}" (id 0) (at 163.7031 90.2494 0)
+      (effects (font (size 1.27 1.27)) (justify left) hide)
     )
   )
@@
     )
   )
-  (global_label "PIN_LEDR" (shape input) (at 187.96 71.12 180) (fields_autoplaced)
-    (effects (font (size 1.27 1.27)) (justify right))
-    (property "Intersheet References" "${INTERSHEET_REFS}" (id 0) (at 176.6569 71.0406 0)
+  (global_label "PIN_LEDR" (shape input) (at 187.96 60.96 180) (fields_autoplaced)
+    (effects (font (size 1.27 1.27)) (justify right))
+    (property "Intersheet References" "${INTERSHEET_REFS}" (id 0) (at 176.6569 61.0394 0)
       (effects (font (size 1.27 1.27)) (justify right) hide)
     )
@@
     )
   )
-  (global_label "PIN_LEDG" (shape input) (at 110.49 71.12 180) (fields_autoplaced)
-    (effects (font (size 1.27 1.27)) (justify right))
-    (property "Intersheet References" "${INTERSHEET_REFS}" (id 0) (at 99.1869 71.0406 0)
-      (effects (font (size 1.27 1.27)) (justify right) hide)
-    )
-  )
-  (global_label "PIN_LEDB" (shape input) (at 110.49 74.93 180) (fields_autoplaced)
-    (effects (font (size 1.27 1.27)) (justify right))
-    (property "Intersheet References" "${INTERSHEET_REFS}" (id 0) (at 99.1869 74.8506 0)
-      (effects (font (size 1.27 1.27)) (justify right) hide)
+  (global_label "PIN_LEDG" (shape input) (at 152.4 86.36 0) (fields_autoplaced)
+    (effects (font (size 1.27 1.27)) (justify left))
+    (property "Intersheet References" "${INTERSHEET_REFS}" (id 0) (at 163.7031 86.4394 0)
+      (effects (font (size 1.27 1.27)) (justify left) hide)
+    )
+  )
+  (global_label "PIN_LEDB" (shape input) (at 152.4 82.55 0) (fields_autoplaced)
+    (effects (font (size 1.27 1.27)) (justify left))
+    (property "Intersheet References" "${INTERSHEET_REFS}" (id 0) (at 163.7031 82.6294 0)
+      (effects (font (size 1.27 1.27)) (justify left) hide)
     )
   )
@@
       (effects (font (size 1.27 1.27)) (justify right))
     )
-    (property "Footprint" "Resistor_SMD:R_0402_1005Metric_Pad0.72x0.64mm_HandSolder" (id 2) (at 50.038 151.13 90)
+    (property "Footprint" "" (id 2) (at 50.038 151.13 90)
       (effects (font (size 1.27 1.27)) hide)
     )
@@
     (property "Reference" "R2" (id 0) (at 44.45 139.7 90))
     (property "Value" "100" (id 1) (at 44.45 142.24 90))
-    (property "Footprint" "Resistor_SMD:R_0402_1005Metric_Pad0.72x0.64mm_HandSolder" (id 2) (at 44.45 146.558 90)
+    (property "Footprint" "" (id 2) (at 44.45 146.558 90)
       (effects (font (size 1.27 1.27)) hide)
     )
@@
     (property "Reference" "B1" (id 0) (at 191.77 71.12 90))
     (property "Value" "R" (id 1) (at 191.77 68.9411 90))
-    (property "Footprint" "Resistor_SMD:R_0402_1005Metric_Pad0.72x0.64mm_HandSolder" (id 2) (at 191.77 69.342 90)
+    (property "Footprint" "" (id 2) (at 191.77 69.342 90)
       (effects (font (size 1.27 1.27)) hide)
     )
@@
     (property "Reference" "G1" (id 0) (at 191.77 66.04 90))
     (property "Value" "R" (id 1) (at 191.77 63.8611 90))
-    (property "Footprint" "Resistor_SMD:R_0402_1005Metric_Pad0.72x0.64mm_HandSolder" (id 2) (at 191.77 64.262 90)
+    (property "Footprint" "" (id 2) (at 191.77 64.262 90)
       (effects (font (size 1.27 1.27)) hide)
     )
@@
     (pin "1")
   )
-  (symbol (lib_id "Device:LED_RKGB") (at 200.66 66.04 180) (unit 1)
-    (in_bom yes) (on_board yes) (fields_autoplaced)
-    (property "Reference" "D2" (id 0) (at 200.66 54.7202 0))
-    (property "Value" "LED_RKGB" (id 1) (at 200.66 57.2571 0))
-    (property "Footprint" "LED_THT:LED_D5.0mm-4_RGB_Wide_Pins" (id 2) (at 200.66 64.77 0)
-      (effects (font (size 1.27 1.27)) hide)
-    )
-    (property "Datasheet" "~" (id 3) (at 200.66 64.77 0)
+  (symbol (lib_id "Device:LED_RKGB") (at 200.66 66.04 0) (mirror y) (unit 1)
+    (in_bom yes) (on_board yes) (fields_autoplaced)
+    (property "Reference" "D2" (id 0) (at 200.66 53.9582 0))
+    (property "Value" "LED_RKGB" (id 1) (at 200.66 56.4951 0))
+    (property "Footprint" "LED_THT:LED_D5.0mm-4_RGB_Wide_Pins" (id 2) (at 200.66 67.31 0)
+      (effects (font (size 1.27 1.27)) hide)
+    )
+    (property "Datasheet" "~" (id 3) (at 200.66 67.31 0)
       (effects (font (size 1.27 1.27)) hide)
     )
@@
     (property "Reference" "R1" (id 0) (at 191.77 60.96 90))
     (property "Value" "R" (id 1) (at 191.77 58.7811 90))
-    (property "Footprint" "Resistor_SMD:R_0402_1005Metric_Pad0.72x0.64mm_HandSolder" (id 2) (at 191.77 59.182 90)
+    (property "Footprint" "" (id 2) (at 191.77 59.182 90)
       (effects (font (size 1.27 1.27)) hide)
     )
@@
     )
     (path "/b7bb8517-00b5-4caf-8c18-eda7de5afdde"
-      (reference "B1") (unit 1) (value "R") (footprint "Resistor_SMD:R_0402_1005Metric_Pad0.72x0.64mm_HandSolder")
+      (reference "B1") (unit 1) (value "R") (footprint "Resistor_SMD:R_1206_3216Metric_Pad1.30x1.75mm_HandSolder")
     )
     (path "/6eb4e5f0-1898-4a31-958e-2e5a03350318"
@@
     )
     (path "/bfd987b2-b471-4edd-9a20-44eb2e980ca7"
-      (reference "G1") (unit 1) (value "R") (footprint "Resistor_SMD:R_0402_1005Metric_Pad0.72x0.64mm_HandSolder")
+      (reference "G1") (unit 1) (value "R") (footprint "Resistor_SMD:R_1206_3216Metric_Pad1.30x1.75mm_HandSolder")
     )
     (path "/2dfbc12a-2aaa-446d-bdb3-48a28cd36745"
@@
     )
     (path "/ed459d60-2755-4580-bbb0-62778a4d08b2"
-      (reference "R1") (unit 1) (value "R") (footprint "Resistor_SMD:R_0402_1005Metric_Pad0.72x0.64mm_HandSolder")
+      (reference "R1") (unit 1) (value "R") (footprint "Resistor_SMD:R_1206_3216Metric_Pad1.30x1.75mm_HandSolder")
     )
     (path "/3b40bec6-88fb-47a7-acdd-0e7fc95b021c"
-      (reference "R2") (unit 1) (value "100") (footprint "Resistor_SMD:R_0402_1005Metric_Pad0.72x0.64mm_HandSolder")
+      (reference "R2") (unit 1) (value "100") (footprint "Resistor_SMD:R_1206_3216Metric_Pad1.30x1.75mm_HandSolder")
     )
     (path "/3b1dc44c-db64-47a9-afdd-0c59a9191aac"
-      (reference "R3") (unit 1) (value "10k") (footprint "Resistor_SMD:R_0402_1005Metric_Pad0.72x0.64mm_HandSolder")
+      (reference "R3") (unit 1) (value "10k") (footprint "Resistor_SMD:R_1206_3216Metric_Pad1.30x1.75mm_HandSolder")
     )
     (path "/1dae53b3-dac4-44f9-bd0e-c8caabe3abc3"

Commit message: Possibly final version of PCB?
Parts:
- B1, G1, R1, R2, R3: footprint (none) -> Resistor_SMD:R_1206_3216Metric_Pad1.30x1.75mm_HandSolder
- Q1: footprint Package_TO_SOT_SMD:SOT-223-3_TabPin2 -> (none)
Connections:
- net GNDS is gone; now on net GND: DIP_MODE1.1, DIP_MODE1.2, DIP_MODE1.3
- net GND: now also BAT1.1 (Pin_1); no longer Q1.3 (S), SW_EN1.3 (C)
- net at Q1.2 (D), SW_EN1.2 (B): now also BAT1.2 (Pin_2); no longer BAT1.1 (Pin_1)
- net BAT+ renamed MCUBAT+
- net MCUBAT+: now also Q1.3 (S), SW_EN1.3 (C); no longer BAT1.2 (Pin_2)
Other:
- moved on the sheet: SW_EN1
