File: footswitch-pcb/footswitch-pcb.kicad_pcb (KiCad board)
At the start: 2 copper layers, 55.9 x 25.4 mm, 6 parts, among them J1 Conn_01x02_Female, J2 Conn_01x02_Female, SW1 SW_LAYER, SW2 SW_BLUETOOTH, SW3 SW_SPST, U1 SeeeduinoXIAO

Commit message: PCB Update
Parts:
- added D1: WS2812B, LED_SMD:LED_WS2812B_PLCC4_5.0x5.0mm_P3.2mm, F.Cu at (149.9, 101.6)
- added D2: LED_RKGB, LED_THT:LED_D5.0mm-4_RGB_Wide_Pins, F.Cu at (162.1, 73.7)
- added J3: Solder_Pad_Reset, TestPoint:TestPoint_Pad_3.0x3.0mm, F.Cu at (119.4, 74.9)
- added J4: Conn_01x02_Male, Connector_JST:JST_XH_S2B-XH-A-1_1x02_P2.50mm_Horizontal, F.Cu at (163.8, 85.1)
- added J5: Solder_Pad_BAT-, TestPoint:TestPoint_Pad_3.0x3.0mm, F.Cu at (153.7, 85.1)
- added R1: R, Resistor_SMD:R_0402_1005Metric_Pad0.72x0.64mm_HandSolder, F.Cu at (168.9, 78.7)
- added R2: R, Resistor_SMD:R_0402_1005Metric_Pad0.72x0.64mm_HandSolder, F.Cu at (166.4, 78.7)
- added R3: R, Resistor_SMD:R_0402_1005Metric_Pad0.72x0.64mm_HandSolder, F.Cu at (162.1, 78.7)
- J1: value Conn_01x02_Female -> Conn_Pedal; footprint Connector_JST:JST_XH_B2B-XH-AM_1x02_P2.50mm_Vertical -> Connector_JST:JST_XH_B2B-XH-A_1x02_P2.50mm_Vertical
- J2: value Conn_01x02_Female -> Solder_Pad_BAT+; footprint Connector_JST:JST_XH_B2B-XH-A_1x02_P2.50mm_Vertical -> TestPoint:TestPoint_Pad_3.0x3.0mm
- SW1: value SW_LAYER -> SW_DIP_x03; footprint Button_Switch_THT:SW_Tactile_SPST_Angled_PTS645Vx39-2LFS -> Button_Switch_THT:SW_DIP_SPSTx03_Slide_6.7x9.18mm_W7.62mm_P2.54mm_LowProfile
- SW3: value SW_SPST -> SW_RESET
- moved SW3 53.1 mm to (109.5, 73.4)
- moved SW2 26.9 mm to (151.4, 73.4)
- moved U1 17.4 mm to (133.3, 81.3)
- moved SW1 17.3 mm to (110.5, 101.6), turned to 90 degrees
- moved J2 10.9 mm to (153.7, 90.2)
- moved J1 1.27 mm to (132.1, 97.8), turned to 0 degrees
Connections:
- J1 pad 1: Net-(U1-Pad5) -> GND
- J1 pad 2: GND -> PIN_PEDAL
- J2 pad 1: Net-(U1-Pad21) -> Net-(J4-Pad2)
- SW1 pad 2: Net-(U1-Pad4) -> GND
- SW2 pad 1: GND -> PIN_BT
- SW2 pad 2: Net-(U1-Pad3) -> GND
- SW3 pad 1: Net-(J2-Pad2) -> Net-(J3-Pad1)
- SW3 pad 2: Net-(U1-Pad22) -> GND
- U1 pad 1: unconnected-(U1-Pad1) -> PIN_BT
- U1 pad 10: unconnected-(U1-Pad10) -> PIN_LAYER2
- U1 pad 11: unconnected-(U1-Pad11) -> PIN_LAYER1
- U1 pad 2: unconnected-(U1-Pad2) -> PIN_LEDR
- U1 pad 21: Net-(U1-Pad21) -> unconnected-(U1-Pad21)
- U1 pad 22: Net-(U1-Pad22) -> unconnected-(U1-Pad22)
- U1 pad 3: Net-(U1-Pad3) -> PIN_LEDG
- U1 pad 4: Net-(U1-Pad4) -> PIN_LEDB
- U1 pad 5: Net-(U1-Pad5) -> unconnected-(U1-Pad5)
- U1 pad 8: unconnected-(U1-Pad8) -> PIN_PEDAL
- U1 pad 9: unconnected-(U1-Pad9) -> PIN_LAYER3
Routing:
- net PIN_LEDB: track 0.00 -> 30.1 mm
- net PIN_LEDG: track 0.00 -> 26.8 mm
- net PIN_LAYER1: track 0.00 -> 24.8 mm
- net Net-(U1-Pad4): track 24.2 -> 0.00 mm
- net PIN_PEDAL: track 0.00 -> 22.3 mm
- net PIN_LEDR: track 0.00 -> 22.1 mm
- net PIN_LAYER2: track 0.00 -> 20.5 mm
- net Net-(J3-Pad1): track 0.00 -> 17.0 mm
- net PIN_LAYER3: track 0.00 -> 16.2 mm
- net Net-(J4-Pad2): track 0.00 -> 15.5 mm
- net Net-(U1-Pad3): track 11.6 -> 0.00 mm
- net Net-(J4-Pad1): track 0.00 -> 10.2 mm
- net PIN_BT: track 0.00 -> 9.66 mm
- net Net-(U1-Pad5): track 7.57 -> 0.00 mm
- net Net-(D2-Pad4): track 0.00 -> 4.64 mm
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Other:
- board outline removed

Commit message: PCB update
Parts:
- removed D1: WS2812B, LED_SMD:LED_WS2812B_PLCC4_5.0x5.0mm_P3.2mm
- SW3: value SW_RESET -> SW_SPDT; footprint Button_Switch_THT:SW_Tactile_SPST_Angled_PTS645Vx39-2LFS -> Button_Switch_THT:SW_Slide_1P2T_CK_OS102011MS2Q
- moved SW3 4.82 mm to (114.3, 73.7)
- moved RST 4.17 mm to (116.8, 78.2), turned to 90 degrees
- moved SW1 3.95 mm to (113.0, 98.5)
- moved SW_BT 2.93 mm to (148.5, 73.7)
- moved Pedal 2.23 mm to (134.2, 97.3), turned to 180 degrees
- moved D2 0.50 mm to (162.1, 74.2)
- moved R1 0.38 mm to (168.5, 78.7)
- renumbered J2 to BAT+, J5 to BAT-, J1 to Pedal, J3 to RST, SW2 to SW_BT
Connections:
- SW3 pad 1: Net-(J3-Pad1) -> unconnected-(SW3-Pad1)
- SW3 pad 2: GND -> Net-(J3-Pad1)
Routing:
- net Net-(J3-Pad1): track 17.0 -> 4.80 mm
- net PIN_LAYER2: track 20.5 -> 15.0 mm
- net PIN_LAYER3: track 16.2 -> 10.6 mm
- net PIN_LAYER1: track 24.8 -> 19.3 mm
- net PIN_BT: track 9.66 -> 6.62 mm
- net PIN_PEDAL: track 22.3 -> 19.3 mm
- net PIN_LEDB: track 30.1 -> 29.2 mm
- net Net-(D2-Pad4): track 4.64 -> 3.98 mm
- net Net-(D2-Pad3): track 4.48 -> 3.98 mm
- net Net-(D2-Pad1): track 4.48 -> 3.98 mm
Other:
- board outline added: 60 x 30 mm

Commit message: PCB Update
Parts:
- removed SW3: SW_SPDT, Button_Switch_THT:SW_Slide_1P2T_CK_OS102011MS2Q
- added BTN_RESET1: BTN_RESET, Button_Switch_THT:SW_PUSH_6mm_H7.3mm, B.Cu at (131.5, 93.7)
- added SW_EN1: SW_ENABLE, Button_Switch_THT:SW_Slide_1P2T_CK_OS102011MS2Q, F.Cu at (114.3, 73.7)
- BTN_BT1: renamed from SW_BT; value SW_BLUETOOTH -> BTN_BLUETOOTH
- DIP_MODE1: renamed from SW1; moved to B.Cu
- Pedal1: renamed from Pedal; footprint Connector_JST:JST_XH_B2B-XH-A_1x02_P2.50mm_Vertical -> Connector_PinHeader_2.54mm:PinHeader_1x02_P2.54mm_Horizontal
- moved RES1 26.1 mm to (135.5, 96.5)
- moved Pedal1 22.8 mm to (119.7, 79.7), turned to -90 degrees
- moved DIP_MODE1 5.20 mm to (118.2, 98.5)
- moved BAT+1 5.17 mm to (148.5, 90.3)
- moved BAT-1 5.17 mm to (148.5, 85.1)
- moved BAT1 2.37 mm to (163.8, 82.7)
- moved B1 1.62 mm to (162.1, 77.1)
- moved R1 1.62 mm to (168.5, 77.1)
- renumbered R3 to B1, BAT+ to BAT+1, BAT- to BAT-1, J4 to BAT1, R2 to G1, RST to RES1
Connections:
- BAT+1 pad 1: Net-(J2-Pad1) -> Net-(BAT+1-Pad1)
- BAT1 pad 2: Net-(J2-Pad1) -> Net-(BAT1-Pad2)
- DIP_MODE1 pad 4: PIN_LAYER3 -> PIN_LAYER1
- DIP_MODE1 pad 6: PIN_LAYER1 -> PIN_LAYER3
- U1 pad 10: PIN_LAYER2 -> PIN_LAYER1
- U1 pad 11: PIN_LAYER1 -> PIN_PEDAL
- U1 pad 8: PIN_PEDAL -> PIN_LAYER3
- U1 pad 9: PIN_LAYER3 -> PIN_LAYER2
Routing:
- net Net-(BAT1-Pad2): track 0.00 -> 75.6 mm
- net Net-(BAT+1-Pad1): track 0.00 -> 55.0 mm, vias 0 -> 1
- net Net-(J2-Pad1): track 15.5 -> 0.00 mm
- net PIN_PEDAL: track 19.3 -> 8.98 mm
- net Net-(BTN_RESET1-Pad1): track 4.80 -> 12.7 mm
- net Net-(BAT-1-Pad1): track 10.2 -> 16.3 mm
- net PIN_LAYER1: track 19.3 -> 14.6 mm
- net PIN_LAYER2: track 15.0 -> 11.1 mm
- net GND: track 3.46 -> 7.17 mm, vias 1 -> 0
- net PIN_LAYER3: track 10.6 -> 7.47 mm
- net PIN_LEDR: track 22.1 -> 23.7 mm
- net Net-(D2-Pad4): track 3.98 -> 2.36 mm
- net Net-(B1-Pad1): track 3.98 -> 2.36 mm
- net PIN_LEDG: track 26.8 -> 26.1 mm
Other:
- outline, holes or cut-outs redrawn
- board text added: "GND"

Commit message: MOSFET?
Parts:
- removed BAT-1: Solder_Pad_BAT-, TestPoint:TestPoint_Pad_3.0x3.0mm
- added Q1: BUK7880-55A, Package_TO_SOT_SMD:SOT-223-3_TabPin2, F.Cu at (157.2, 87.9)
- added R2: 100, Resistor_SMD:R_0402_1005Metric_Pad0.72x0.64mm_HandSolder, F.Cu at (147.7, 91.9)
- added R3: 10k, Resistor_SMD:R_0402_1005Metric_Pad0.72x0.64mm_HandSolder, F.Cu at (151.7, 91.9)
- BAT1: value Conn_01x02_Male -> Battery Connector
- moved BAT+1 6.44 mm to (150.4, 84.1)
Connections:
- BAT+1 pad 1: Net-(BAT+1-Pad1) -> Net-(BAT1-Pad2)
- BAT1 pad 1: Net-(BAT-1-Pad1) -> GNDS
- DIP_MODE1 pad 1: GND -> GNDS
- DIP_MODE1 pad 2: GND -> GNDS
- DIP_MODE1 pad 3: GND -> GNDS
- SW_EN1 pad 2: Net-(BAT+1-Pad1) -> GNDS
- SW_EN1 pad 3: Net-(BAT1-Pad2) -> GND
- U1 pad 14: unconnected-(U1-Pad14) -> 5V_USB
Routing:
- net GNDS: track 0.00 -> 99.5 mm
- net Net-(BAT+1-Pad1): track 55.0 -> 0.00 mm, vias 1 -> 0
- net Net-(BAT1-Pad2): track 75.6 -> 21.4 mm, vias 0 -> 1
- net 5V_USB: track 0.00 -> 45.5 mm, vias 0 -> 2
- net Net-(BAT-1-Pad1): track 16.3 -> 0.00 mm
- net GND: track 7.17 -> 21.9 mm, vias 0 -> 2
- net Net-(Q1-Pad1): track 0.00 -> 7.30 mm
Other:
- board text added: "- +"

Commit message: THT Pogo Pins
Parts:
- removed BAT+1: Solder_Pad_BAT+, TestPoint:TestPoint_Pad_3.0x3.0mm
- removed RES1: Solder_Pad_Reset, TestPoint:TestPoint_Pad_3.0x3.0mm
- moved R1 47.4 mm to (121.2, 79.3), turned to 180 degrees
- moved G1 45.2 mm to (121.2, 76.8), turned to 180 degrees
- moved D2 43.6 mm to (118.4, 75.1), turned to 180 degrees
- moved B1 41.0 mm to (121.2, 74.2), turned to 0 degrees
- moved SW_EN1 33.8 mm to (148.1, 73.2)
- moved BTN_BT1 14.1 mm to (162.6, 73.7)
- moved R2 7.78 mm to (147.1, 84.1)
- moved Q1 5.69 mm to (153.1, 83.9)
- moved Pedal1 3.13 mm to (119.6, 82.8)
- moved R3 1.61 mm to (153.2, 91.2), turned to 180 degrees
- moved BAT1 0.67 mm to (163.6, 83.4)
- moved U1 0.55 mm to (133.3, 81.8)
Connections:
- BAT1 pad 1: GNDS -> Net-(BAT1-Pad1)
- BAT1 pad 2: Net-(BAT1-Pad2) -> BAT+
- BTN_RESET1 pad 1: Net-(BTN_RESET1-Pad1) -> RESET
- G1 pad 1: Net-(D2-Pad3) -> PIN_LEDG
- G1 pad 2: PIN_LEDG -> Net-(D2-Pad3)
- Q1 pad 2: GNDS -> Net-(BAT1-Pad1)
- R1 pad 1: Net-(D2-Pad4) -> PIN_LEDB
- R1 pad 2: PIN_LEDB -> Net-(D2-Pad4)
- R2 pad 1: 5V_USB -> Net-(Q1-Pad1)
- R2 pad 2: Net-(Q1-Pad1) -> 5V_USB
- SW_EN1 pad 2: GNDS -> Net-(BAT1-Pad1)
- U1 pad 1: PIN_BT -> PIN_LEDR
- U1 pad 10: PIN_LAYER1 -> unconnected-(U1-Pad10)
- U1 pad 11: PIN_PEDAL -> PIN_BT
- U1 pad 2: PIN_LEDR -> PIN_LEDG
- U1 pad 3: PIN_LEDG -> PIN_LEDB
- U1 pad 4: PIN_LEDB -> PIN_PEDAL
- U1 pad 5: unconnected-(U1-Pad5) -> PIN_LAYER1
- U1 pad 6: unconnected-(U1-Pad6) -> PIN_LAYER2
- U1 pad 7: unconnected-(U1-Pad7) -> PIN_LAYER3
- U1 pad 8: PIN_LAYER3 -> unconnected-(U1-Pad8)
- U1 pad 9: PIN_LAYER2 -> unconnected-(U1-Pad9)
Routing:
- net GNDS: track 99.5 -> 0.00 mm
- net BAT+: track 0.00 -> 50.5 mm
- net 5V_USB: track 45.5 -> 12.7 mm, vias 2 -> 0
- net Net-(BAT1-Pad1): track 0.00 -> 27.2 mm
- net PIN_LEDB: track 29.1 -> 3.95 mm
- net RESET: track 0.00 -> 24.4 mm
- net PIN_BT: track 6.62 -> 29.1 mm
- net PIN_LEDG: track 26.1 -> 3.95 mm
- net Net-(BAT1-Pad2): track 21.4 -> 0.00 mm, vias 1 -> 0
- net PIN_LEDR: track 23.7 -> 3.95 mm
- net GND: track 21.9 -> 4.82 mm, vias 2 -> 1
- net Net-(BTN_RESET1-Pad1): track 12.7 -> 0.00 mm
- net Net-(D2-Pad4): track 2.36 -> 10.4 mm
- net Net-(D2-Pad3): track 3.98 -> 7.16 mm
- net Net-(Q1-Pad1): track 7.30 -> 10.3 mm
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Other:
- outline, holes or cut-outs redrawn

Commit message: v3
Parts:
- B1, G1, R1, R2, R3: footprint Resistor_SMD:R_0402_1005Metric_Pad0.72x0.64mm_HandSolder -> Resistor_SMD:R_1206_3216Metric_Pad1.30x1.75mm_HandSolder
- moved D2 49.7 mm to (168.1, 75.0)
- moved BAT1 49.3 mm to (115.1, 91.9)
- moved DIP_MODE1 45.5 mm to (160.5, 81.8), turned to -90 degrees
- moved Pedal1 38.1 mm to (154.9, 97.3), turned to 180 degrees
- moved BTN_RESET1 34.9 mm to (166.4, 92.7)
- moved SW_EN1 34.3 mm to (113.8, 73.7)
- moved R2 34.1 mm to (113.0, 85.1), turned to 180 degrees
- moved Q1 34.0 mm to (119.1, 81.8)
- moved R3 30.5 mm to (122.7, 90.0), turned to -90 degrees
- moved G1 29.8 mm to (149.2, 86.9), turned to 0 degrees
- moved R1 29.8 mm to (149.2, 89.4), turned to 0 degrees
- moved B1 29.8 mm to (149.2, 84.3), turned to 180 degrees
- moved BTN_BT1 13.7 mm to (148.9, 73.9)
- moved U1 2.54 mm to (135.9, 81.8)
Connections:
- B1 pad 2: PIN_LEDR -> PIN_LEDB
- D2 pad 1: Net-(B1-Pad1) -> Net-(D2-Pad1)
- D2 pad 4: Net-(D2-Pad4) -> Net-(B1-Pad1)
- R1 pad 1: PIN_LEDB -> PIN_LEDR
- R1 pad 2: Net-(D2-Pad4) -> Net-(D2-Pad1)
- U1 pad 1: PIN_LEDR -> unconnected-(U1-Pad1)
- U1 pad 10: unconnected-(U1-Pad10) -> PIN_LEDB
- U1 pad 2: PIN_LEDG -> unconnected-(U1-Pad2)
- U1 pad 3: PIN_LEDB -> unconnected-(U1-Pad3)
- U1 pad 8: unconnected-(U1-Pad8) -> PIN_LEDR
- U1 pad 9: unconnected-(U1-Pad9) -> PIN_LEDG
Routing:
- net GND: track 4.82 -> 41.9 mm, vias 1 -> 0
- net PIN_PEDAL: track 9.21 -> 43.1 mm, vias 0 -> 1
- net 5V_USB: track 12.7 -> 40.1 mm, vias 0 -> 1
- net PIN_LAYER3: track 8.59 -> 35.8 mm
- net Net-(D2-Pad1): track 0.00 -> 27.0 mm
- net PIN_LAYER2: track 12.4 -> 39.2 mm
- net PIN_LAYER1: track 16.6 -> 43.0 mm
- net RESET: track 24.4 -> 43.6 mm
- net PIN_BT: track 29.1 -> 11.8 mm
- net BAT+: track 50.5 -> 35.3 mm
- net Net-(B1-Pad1): track 2.54 -> 16.6 mm
- net Net-(D2-Pad3): track 7.16 -> 20.8 mm
- net Net-(D2-Pad4): track 10.4 -> 0.00 mm
- net Net-(BAT1-Pad1): track 27.2 -> 22.1 mm
- net Net-(Q1-Pad1): track 10.3 -> 12.5 mm, vias 0 -> 2
Other:
- outline, holes or cut-outs redrawn
- board text removed: "- +"

Commit message: Possibly final version of PCB?
Parts:
- Q1: footprint Package_TO_SOT_SMD:SOT-223-3_TabPin2 -> Package_TO_SOT_SMD:SOT-23
- moved BTN_RESET1 33.4 mm to (135.9, 78.9), turned to -90 degrees
- moved R2 28.4 mm to (139.2, 74.1), turned to 0 degrees
- moved R3 17.4 mm to (138.2, 82.1), turned to 180 degrees
- moved Pedal1 15.6 mm to (156.6, 81.8), turned to -90 degrees
- moved Q1 14.5 mm to (132.2, 88.1)
- moved BAT1 11.6 mm to (120.8, 81.8)
- moved SW_EN1 3.67 mm to (117.5, 73.7)
- moved BTN_BT1 1.24 mm to (147.6, 73.9)
Connections:
- BAT1 pad 1: Net-(BAT1-Pad1) -> GND
- BAT1 pad 2: BAT+ -> Net-(BAT1-Pad2)
- DIP_MODE1 pad 1: GNDS -> GND
- DIP_MODE1 pad 2: GNDS -> GND
- DIP_MODE1 pad 3: GNDS -> GND
- Q1 pad 2: Net-(BAT1-Pad1) -> Net-(BAT1-Pad2)
- Q1 pad 3: GND -> MCUBAT+
- SW_EN1 pad 2: Net-(BAT1-Pad1) -> Net-(BAT1-Pad2)
- SW_EN1 pad 3: GND -> MCUBAT+
- U1 pad 22: BAT+ -> MCUBAT+
Routing:
- net 5V_USB: track 40.1 -> 2.80 mm, vias 1 -> 0
- net BAT+: track 35.3 -> 0.00 mm
- net RESET: track 43.6 -> 10.6 mm
- net Net-(BAT1-Pad2): track 0.00 -> 29.7 mm, vias 0 -> 1
- net MCUBAT+: track 0.00 -> 29.5 mm
- net Net-(BAT1-Pad1): track 22.1 -> 0.00 mm
- net Net-(Q1-Pad1): track 12.5 -> 27.8 mm, vias 2 -> 0
- net GND: track 41.9 -> 27.6 mm
- net PIN_PEDAL: track 43.1 -> 44.6 mm, vias 1 -> 0
- net PIN_LAYER3: track 35.8 -> 35.0 mm
- net PIN_BT: track 11.8 -> 11.1 mm
Other:
- board size 60 x 30 mm -> 56 x 22 mm
- board text removed: "GND"

Commit message: v1.0?
Parts:
- added G***: LOGO, footswitch-pcb:bass_clave, F.Cu at (116.1, 86.6)
- added G***: LOGO, footswitch-pcb:repo-qr-small, F.Cu at (163.1, 85.6)
- added G***: LOGO, footswitch-pcb:bass_clave, B.Cu at (149.8, 85.6)
- added G***: LOGO, footswitch-pcb:repo-qr, B.Cu at (118.8, 88.1)
- - BATTERY +: renamed from BAT1
- moved SW_POWER 0.36 mm to (117.8, 73.7)
- moved BTN_RESET 0.33 mm to (135.6, 78.9)
- renumbered B1 to B, BTN_BT1 to BTN_BT, BTN_RESET1 to BTN_RESET, DIP_MODE1 to DIP_MODE, G1 to G, Pedal1 to Pedal, R1 to R, SW_EN1 to SW_POWER
Routing:
- net RESET: track 10.6 -> 9.84 mm
Other:
- board text added: "github.com/4cello/FlipStompBLE"
- board text added: "v1.0"
